File: hardware/slice_template.kicad_sch (KiCad schematic)
At the start: 19 parts, among them J1 Conn_01x10_Socket, SW1 SW_DIP_x04, U1 AP63205

Commit message: fix: clear erc/drc errors
Changed lines of the file:
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@@
+	)
+	(junction
+		(at 289.56 200.66)
+		(diameter 0)
+		(color 0 0 0 0)
 	)
 	(junction
@@
 	)
 	(junction
-		(at 289.56 196.85)
-		(diameter 0)
-		(color 0 0 0 0)
-	)
-	(junction
 		(at 99.06 147.32)
 		(diameter 0)
@@
 	(wire
 		(pts
-			(xy 240.03 196.85) (xy 289.56 196.85)
+			(xy 240.03 200.66) (xy 289.56 200.66)
 		)
 		(stroke
@@
 	(wire
 		(pts
+			(xy 289.56 157.48) (xy 289.56 200.66)
+		)
+		(stroke
+			(width 0.2032)
+			(type default)
+			(color 0 0 0 1)
+		)
+	)
+	(wire
+		(pts
 			(xy 250.19 116.84) (xy 266.7 116.84)
 		)
@@
 	(wire
 		(pts
-			(xy 289.56 196.85) (xy 332.74 196.85)
+			(xy 289.56 200.66) (xy 332.74 200.66)
 		)
 		(stroke
@@
 	(wire
 		(pts
-			(xy 240.03 147.32) (xy 240.03 196.85)
+			(xy 240.03 147.32) (xy 240.03 200.66)
 		)
 		(stroke
@@
 			(type default)
 			(color 221 133 0 1)
-		)
-	)
-	(wire
-		(pts
-			(xy 289.56 157.48) (xy 289.56 196.85)
-		)
-		(stroke
-			(width 0.2032)
-			(type default)
-			(color 0 0 0 1)
 		)
 	)
@@
 	(hierarchical_label "GND"
 		(shape input)
-		(at 332.74 196.85 0)
-		(effects
-			(font
+		(at 332.74 200.66 0)
+		(effects
+			(font
